Commit message: pigeon files

File: pigeon/pigeon.URDF (robot description, URDF)
Before this commit: robot pigeon, 30 links, 29 joints
Links:
- link left_fingers: geometry visual mesh filename=meshes/fingers_texture.STL
- link left_hand_wing: geometry visual mesh filename=meshes/left_hand_wing_texture.STL
- link left_lower_leg: geometry visual mesh filename=meshes/lower_leg_texture.STL
- link left_mid_leg: geometry visual mesh filename=meshes/mid_leg_texture.STL
- link left_mid_wing: geometry visual mesh filename=meshes/left_mid_wing_texture.STL
- link left_thumb: geometry visual mesh filename=meshes/thumb_texture.STL
- link left_upper_leg: geometry visual mesh filename=meshes/upper_leg_texture.STL
- link left_upper_wing: geometry visual mesh filename=meshes/left_upper_wing_texture.STL
- link right_fingers: geometry visual mesh filename=meshes/fingers_texture.STL
- link right_hand_wing: geometry visual mesh filename=meshes/left_hand_wing_texture.STL
- link right_lower_leg: geometry visual mesh filename=meshes/lower_leg_texture.STL
- link right_mid_leg: geometry visual mesh filename=meshes/mid_leg_texture.STL
- link right_mid_wing: geometry visual mesh filename=meshes/left_mid_wing_texture.STL
- link right_thumb: geometry visual mesh filename=meshes/thumb_texture.STL
- link right_upper_leg: geometry visual mesh filename=meshes/upper_leg_texture.STL
- link right_upper_wing: geometry visual mesh filename=meshes/left_upper_wing_texture.STL
- link tail: geometry visual mesh filename=meshes/tail_texture.STL
- link torso: geometry visual mesh filename=meshes/torso_texture.STL
